File: Alchitry_HDMI_Shield/Alchitry_HDMI_Shield.kicad_pcb (KiCad board)
At the start: 2 copper layers, 65 x 45 mm, 26 parts, among them J1 HDMI_A_1.4, U1 boardmezzanine_new, U3 TFP410

Commit message: both shift not working
Parts:
- J1: footprint Connector_HDMI:HDMI_Jing_C168714 -> Custom_Parts:HDMI
- U1: footprint alchitry:ELEMENT -> Custom_Parts:Alchitry_Top_Bottom
Routing:
- net GNDREF: vias 65 -> 69
