File: Alchitry_HDMI_Shield/V2Alchitry_HDMI_Shield copy.kicad_pcb (KiCad board)
At the start: 2 copper layers, 65 x 45 mm, 26 parts, among them J1 HDMI_A_1.4, U3 TFP410

Commit message: both shift not working
Parts:
- J1: footprint Connector_HDMI:HDMI_Jing_C168714 -> Custom_Parts:HDMI
- REF**: value ELEMENT -> Alchitry_Top_Bottom; footprint alchitry:ELEMENT -> Custom_Parts:Alchitry_Top_Bottom
