File: Alchitry_IO_Shield_TFP410 - V2/LEDs.sch (KiCad schematic (older format))
At the start: 39 parts, among them SW1 SW_DIP_x08, SW2 SW_DIP_x08, SW3 SW_DIP_x08

Commit message: update to shield
Parts:
- added AFF1, AFF2, AFF3, AFF4: LTS-6960HR, Display_7Segment:KCSC02-136, symbol Display_Character:LTS-6960HR
- added Q1, Q2, Q3, Q4: Q_PMOS_SGD, Package_TO_SOT_SMD:SOT-23, symbol Device:Q_PMOS_GSD
- added RN14, RN15, RN16, RN17, RN18, RN19, RN20, RN21: R_Pack04, Resistor_SMD:R_Array_Convex_4x0603, symbol Device:R_Pack04
Connections:
- net labels added: +3V3, AN0, AN1, AN2, AN3, AN[0..3], C0, C1, C2, C3, C4, C5, C6, C[0..6], DP
- wire segments 288 -> 340
