File: Alchitry_IO_Shield_TFP410 - V5/KiCad Project Files/7Seg_Btns.kicad_sch (KiCad schematic)
At the start: 13 parts, among them Q1 NTZD3152P, Q2 NTZD3152P, SW1 SW3, SW2 SW1, SW3 SW2, SW4 SW4, U3 0402_7Seg_CA, U4 0402_7Seg_CA, U5 0402_7Seg_CA, U6 0402_7Seg_CA

Commit message: laid out switches, btns and leds
Parts:
- renumbered Q1 to Q3, Q2 to Q4, RN2 to RN3, SW1 to SW5, SW2 to SW6, SW3 to SW7, SW4 to SW8, U6 to U10, U3 to U7, U4 to U8, U5 to U9
Changed lines of the file:
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@@
   (symbol (lib_id "power:+3V3") (at 78.105 77.47 0)
     (in_bom yes) (on_board yes)
-    (property "Reference" "#PWR0106" (id 0) (at 78.105 81.28 0)
+    (property "Reference" "#PWR0114" (id 0) (at 78.105 81.28 0)
       (effects (font (size 1.27 1.27)) hide)
     )
@@
   (symbol (lib_id "power:+3V3") (at 136.525 77.47 0)
     (in_bom yes) (on_board yes)
-    (property "Reference" "#PWR0104" (id 0) (at 136.525 81.28 0)
+    (property "Reference" "#PWR0112" (id 0) (at 136.525 81.28 0)
       (effects (font (size 1.27 1.27)) hide)
     )
@@
   (symbol (lib_id "power:+3V3") (at 151.13 129.54 0)
     (in_bom yes) (on_board yes)
-    (property "Reference" "#PWR0111" (id 0) (at 151.13 133.35 0)
+    (property "Reference" "#PWR0119" (id 0) (at 151.13 133.35 0)
       (effects (font (size 1.27 1.27)) hide)
     )
@@
   (symbol (lib_id "power:+3V3") (at 165.1 129.54 0)
     (in_bom yes) (on_board yes)
-    (property "Reference" "#PWR0109" (id 0) (at 165.1 133.35 0)
+    (property "Reference" "#PWR0117" (id 0) (at 165.1 133.35 0)
       (effects (font (size 1.27 1.27)) hide)
     )
@@
   (symbol (lib_id "power:+3V3") (at 176.53 129.54 0)
     (in_bom yes) (on_board yes)
-    (property "Reference" "#PWR0110" (id 0) (at 176.53 133.35 0)
+    (property "Reference" "#PWR0118" (id 0) (at 176.53 133.35 0)
       (effects (font (size 1.27 1.27)) hide)
     )
@@
   (symbol (lib_id "power:+3V3") (at 197.485 77.47 0)
     (in_bom yes) (on_board yes)
-    (property "Reference" "#PWR0107" (id 0) (at 197.485 81.28 0)
+    (property "Reference" "#PWR0115" (id 0) (at 197.485 81.28 0)
       (effects (font (size 1.27 1.27)) hide)
     )
@@
   (symbol (lib_id "power:+3V3") (at 258.445 77.47 0)
     (in_bom yes) (on_board yes)
-    (property "Reference" "#PWR0108" (id 0) (at 258.445 81.28 0)
+    (property "Reference" "#PWR0116" (id 0) (at 258.445 81.28 0)
       (effects (font (size 1.27 1.27)) hide)
     )
@@
   (symbol (lib_id "power:GNDREF") (at 153.67 178.435 0)
     (in_bom yes) (on_board yes)
-    (property "Reference" "#PWR0105" (id 0) (at 153.67 184.785 0)
+    (property "Reference" "#PWR0113" (id 0) (at 153.67 184.785 0)
       (effects (font (size 1.27 1.27)) hide)
     )
@@
   (symbol (lib_id "Switch:SW_Push_45deg") (at 148.59 142.24 90)
     (in_bom yes) (on_board yes)
-    (property "Reference" "SW1" (id 0) (at 152.1461 141.0906 90)
+    (property "Reference" "SW5" (id 0) (at 152.1461 141.0906 90)
       (effects (font (size 1.27 1.27)) (justify right))
     )
@@
   (symbol (lib_id "Switch:SW_Push_45deg") (at 162.56 134.62 90)
     (in_bom yes) (on_board yes)
-    (property "Reference" "SW2" (id 0) (at 166.1161 133.4706 90)
+    (property "Reference" "SW6" (id 0) (at 166.1161 133.4706 90)
       (effects (font (size 1.27 1.27)) (justify right))
     )
@@
   (symbol (lib_id "Switch:SW_Push_45deg") (at 162.56 151.13 90)
     (in_bom yes) (on_board yes)
-    (property "Reference" "SW3" (id 0) (at 166.1161 149.9806 90)
+    (property "Reference" "SW7" (id 0) (at 166.1161 149.9806 90)
       (effects (font (size 1.27 1.27)) (justify right))
     )
@@
   (symbol (lib_id "Switch:SW_Push_45deg") (at 173.99 142.24 90)
     (in_bom yes) (on_board yes)
-    (property "Reference" "SW4" (id 0) (at 177.5461 141.0906 90)
+    (property "Reference" "SW8" (id 0) (at 177.5461 141.0906 90)
       (effects (font (size 1.27 1.27)) (justify right))
     )
@@
   (symbol (lib_id "Custom_Transistors:NTZD3152P") (at 78.105 82.55 0)
     (in_bom yes) (on_board yes)
-    (property "Reference" "Q1" (id 0) (at 81.915 80.645 0)
+    (property "Reference" "Q3" (id 0) (at 81.915 80.645 0)
       (effects (font (size 1.27 1.27)) (justify left))
     )
@@
   (symbol (lib_id "Custom_Transistors:NTZD3152P") (at 136.525 82.55 0)
     (in_bom yes) (on_board yes)
-    (property "Reference" "Q1" (id 0) (at 139.7 81.28 0)
+    (property "Reference" "Q3" (id 0) (at 139.7 81.28 0)
       (effects (font (size 1.27 1.27)) (justify left))
     )
@@
   (symbol (lib_id "Custom_Transistors:NTZD3152P") (at 197.485 82.55 0)
     (in_bom yes) (on_board yes)
-    (property "Reference" "Q2" (id 0) (at 201.295 80.645 0)
+    (property "Reference" "Q4" (id 0) (at 201.295 80.645 0)
       (effects (font (size 1.27 1.27)) (justify left))
     )
@@
   (symbol (lib_id "Custom_Transistors:NTZD3152P") (at 258.445 82.55 0)
     (in_bom yes) (on_board yes)
-    (property "Reference" "Q2" (id 0) (at 262.255 80.645 0)
+    (property "Reference" "Q4" (id 0) (at 262.255 80.645 0)
       (effects (font (size 1.27 1.27)) (justify left))
     )
@@
   (symbol (lib_name "Device:R_Pack04_1") (lib_id "Device:R_Pack04") (at 152.4 166.37 180)
     (in_bom yes) (on_board yes)
-    (property "Reference" "RN2" (id 0) (at 147.6248 167.5384 0)
+    (property "Reference" "RN3" (id 0) (at 147.6248 167.5384 0)
       (effects (font (size 1.27 1.27)) (justify left))
     )
@@
   (symbol (lib_id "Custom_LEDs:0402_7Seg_CA_W_Res") (at 64.77 102.235 0)
     (in_bom yes) (on_board yes)
-    (property "Reference" "U3" (id 0) (at 66.04 84.455 0))
+    (property "Reference" "U7" (id 0) (at 66.04 84.455 0))
     (property "Value" "0402_7Seg_CA" (id 1) (at 66.04 86.995 0))
     (property "Footprint" "Custom_LEDs:0402_7Seg_CA_W_Res" (id 2) (at 52.07 119.38 0)
@@
   (symbol (lib_id "Custom_LEDs:0402_7Seg_CA_W_Res") (at 123.19 102.235 0)
     (in_bom yes) (on_board yes)
-    (property "Reference" "U4" (id 0) (at 124.46 84.455 0))
+    (property "Reference" "U8" (id 0) (at 124.46 84.455 0))
     (property "Value" "0402_7Seg_CA" (id 1) (at 124.46 86.995 0))
     (property "Footprint" "Custom_LEDs:0402_7Seg_CA_W_Res" (id 2) (at 110.49 119.38 0)
@@
   (symbol (lib_name "Custom_LEDs:0402_7Seg_CA_1") (lib_id "Custom_LEDs:0402_7Seg_CA_W_Res") (at 184.15 102.235 0)
     (in_bom yes) (on_board yes)
-    (property "Reference" "U5" (id 0) (at 185.42 84.455 0))
+    (property "Reference" "U9" (id 0) (at 185.42 84.455 0))
     (property "Value" "0402_7Seg_CA" (id 1) (at 185.42 86.995 0))
     (property "Footprint" "Custom_LEDs:0402_7Seg_CA_W_Res" (id 2) (at 171.45 119.38 0)
@@
   (symbol (lib_id "Custom_LEDs:0402_7Seg_CA_W_Res") (at 245.11 102.235 0)
     (in_bom yes) (on_board yes)
-    (property "Reference" "U6" (id 0) (at 246.38 84.455 0))
+    (property "Reference" "U10" (id 0) (at 246.38 84.455 0))
     (property "Value" "0402_7Seg_CA" (id 1) (at 246.38 86.995 0))
     (property "Footprint" "Custom_LEDs:0402_7Seg_CA_W_Res" (id 2) (at 232.41 119.38 0)
