File: IO_Shield_W_HDMI/Alchitry_IO_Shield_TFP410 - V4/KiCad Project Files/Alchitry_IO_Shield.kicad_pcb (KiCad board)
At the start: 4 copper layers, 65 x 45 mm, 66 parts, among them J0 HDMI_A_1.4, Q1 Q_PMOS_SGD, Q2 Q_PMOS_SGD, Q3 Q_PMOS_SGD, SW1 SW_DIP_x08, SW2 SW_DIP_x08, U0 boardmezzanine_new, U1 TFP410

Commit message: LOGO ADDED
Parts:
- added G***: LOGO, Logo_Schem&PCB:Ayeeditya_PCB_Logo_Solder_Mask, F.Cu at (20.0, 18.0)
Other:
- board text removed: "AYEEDITYA"

Commit message: Starting a play shield layout
Parts:
- added G***: LOGO, Logo_Schem&PCB:Ayeeditya_PCB_Logo_Solder_Mask_Silk, B.Cu at (42.8, 35.0)
Routing:
- net +3V3: track 117.4 -> 121.0 mm
Other:
- net class Default removed
- net class pwr removed
- board text added: "IO shield + HDMI V4.0"

Commit message: minor changes
Parts:
- removed G***: LOGO, Logo_Schem&PCB:Ayeeditya_PCB_Logo_Solder_Mask_Silk
- removed G***: LOGO, Logo_Schem&PCB:Ayeeditya_PCB_Logo_Solder_Mask
- renumbered DK1 to JP1, DK2 to JP2, DK3 to JP3, DKEN to JP4
Connections:
- J0 pad 18: Net-(J0-Pad18) -> +3V3
- JP0 pad 2: Net-(J0-Pad18) -> +3V3
Routing:
- net GNDREF: track 166.2 -> 115.7 mm, vias 63 -> 39
- net +3V3: track 121.0 -> 73.5 mm, vias 58 -> 35
- net Net-(J0-Pad18): track 7.34 -> 0.00 mm, vias 1 -> 0
- net Net-(AFF3-Pad3): track 32.8 -> 31.9 mm
- net /C1: track 76.9 -> 76.0 mm, vias 6 -> 5
- net /DIP14: track 25.4 -> 24.8 mm
Other:
- board text added: "ADSEHGAL IO shield + HDMI V4.0"
- board text removed: "IO shield + HDMI V4.0"

Commit message: updated shield v4 schematic
Parts:
- added G***: LOGO, LOGO, F.Cu at (21.0, 17.0)
- C1: renamed from C0; footprint Capacitor_SMD:C_0603_1608Metric_Pad1.05x0.95mm_HandSolder -> Capacitor_SMD:C_0603_1608Metric
- C2: renamed from C1; footprint Capacitor_SMD:C_0603_1608Metric_Pad1.05x0.95mm_HandSolder -> Capacitor_SMD:C_0603_1608Metric
- C3: renamed from C2; footprint Capacitor_SMD:C_0603_1608Metric_Pad1.05x0.95mm_HandSolder -> Capacitor_SMD:C_0603_1608Metric
- C4: renamed from C7; footprint Capacitor_SMD:C_0603_1608Metric_Pad1.05x0.95mm_HandSolder -> Capacitor_SMD:C_0603_1608Metric
- D1: renamed from D0; footprint LED_SMD:LED_0603_1608Metric_Pad1.05x0.95mm_HandSolder -> LED_SMD:LED_0603_1608Metric
- D10: renamed from D9; footprint LED_SMD:LED_0603_1608Metric_Pad1.05x0.95mm_HandSolder -> LED_SMD:LED_0603_1608Metric
- D11: renamed from D10; footprint LED_SMD:LED_0603_1608Metric_Pad1.05x0.95mm_HandSolder -> LED_SMD:LED_0603_1608Metric
- D12: renamed from D11; footprint LED_SMD:LED_0603_1608Metric_Pad1.05x0.95mm_HandSolder -> LED_SMD:LED_0603_1608Metric
- D13: renamed from D12; footprint LED_SMD:LED_0603_1608Metric_Pad1.05x0.95mm_HandSolder -> LED_SMD:LED_0603_1608Metric
- D14: renamed from D13; footprint LED_SMD:LED_0603_1608Metric_Pad1.05x0.95mm_HandSolder -> LED_SMD:LED_0603_1608Metric
- D15: renamed from D14; footprint LED_SMD:LED_0603_1608Metric_Pad1.05x0.95mm_HandSolder -> LED_SMD:LED_0603_1608Metric
- D16: renamed from D15; footprint LED_SMD:LED_0603_1608Metric_Pad1.05x0.95mm_HandSolder -> LED_SMD:LED_0603_1608Metric
- D17: renamed from D16; footprint LED_SMD:LED_0603_1608Metric_Pad1.05x0.95mm_HandSolder -> LED_SMD:LED_0603_1608Metric
- D18: renamed from D17; footprint LED_SMD:LED_0603_1608Metric_Pad1.05x0.95mm_HandSolder -> LED_SMD:LED_0603_1608Metric
- D19: renamed from D18; footprint LED_SMD:LED_0603_1608Metric_Pad1.05x0.95mm_HandSolder -> LED_SMD:LED_0603_1608Metric
- D2: renamed from D1; footprint LED_SMD:LED_0603_1608Metric_Pad1.05x0.95mm_HandSolder -> LED_SMD:LED_0603_1608Metric
- D20: renamed from D19; footprint LED_SMD:LED_0603_1608Metric_Pad1.05x0.95mm_HandSolder -> LED_SMD:LED_0603_1608Metric
- D21: renamed from D20; footprint LED_SMD:LED_0603_1608Metric_Pad1.05x0.95mm_HandSolder -> LED_SMD:LED_0603_1608Metric
- D22: renamed from D21; footprint LED_SMD:LED_0603_1608Metric_Pad1.05x0.95mm_HandSolder -> LED_SMD:LED_0603_1608Metric
- D23: renamed from D22; footprint LED_SMD:LED_0603_1608Metric_Pad1.05x0.95mm_HandSolder -> LED_SMD:LED_0603_1608Metric
- D24: renamed from D23; footprint LED_SMD:LED_0603_1608Metric_Pad1.05x0.95mm_HandSolder -> LED_SMD:LED_0603_1608Metric
- D3: renamed from D2; footprint LED_SMD:LED_0603_1608Metric_Pad1.05x0.95mm_HandSolder -> LED_SMD:LED_0603_1608Metric
- D4: renamed from D3; footprint LED_SMD:LED_0603_1608Metric_Pad1.05x0.95mm_HandSolder -> LED_SMD:LED_0603_1608Metric
- D5: renamed from D4; footprint LED_SMD:LED_0603_1608Metric_Pad1.05x0.95mm_HandSolder -> LED_SMD:LED_0603_1608Metric
- D6: renamed from D5; footprint LED_SMD:LED_0603_1608Metric_Pad1.05x0.95mm_HandSolder -> LED_SMD:LED_0603_1608Metric
- D7: renamed from D6; footprint LED_SMD:LED_0603_1608Metric_Pad1.05x0.95mm_HandSolder -> LED_SMD:LED_0603_1608Metric
- D8: renamed from D7; footprint LED_SMD:LED_0603_1608Metric_Pad1.05x0.95mm_HandSolder -> LED_SMD:LED_0603_1608Metric
- D9: renamed from D8; footprint LED_SMD:LED_0603_1608Metric_Pad1.05x0.95mm_HandSolder -> LED_SMD:LED_0603_1608Metric
- R1: renamed from R0; footprint Resistor_SMD:R_0603_1608Metric_Pad1.05x0.95mm_HandSolder -> Resistor_SMD:R_0603_1608Metric
- R3: renamed from R2; moved to F.Cu
- moved RN1 2.00 mm to (24.6, 54.9)
- moved R3 1.56 mm to (18.0, 53.5), turned to 90 degrees
- moved JP2 0.99 mm to (28.8, 43.4)
- moved R2 0.80 mm to (21.2, 51.4)
- moved R1 0.80 mm to (21.2, 48.4)
- moved JP5 0.67 mm to (24.5, 43.4)
- moved R4 0.50 mm to (29.5, 52.8)
- moved JP3 0.40 mm to (30.6, 46.6)
- moved JP4 0.40 mm to (30.6, 50.0)
- moved C4 0.35 mm to (31.9, 54.5)
- moved R5 0.10 mm to (32.6, 52.8)
- renumbered J0 to J1, JP0 to JP1, JP1 to JP2, JP2 to JP3, JP3 to JP4, JP4 to JP5, R1 to R2, R3 to R4, R4 to R5, RN7 to RN1, RN5 to RN10, RN6 to RN11, RN18 to RN12, RN20 to RN13, RN8 to RN14, RN9 to RN15, RN10 to RN16, RN11 to RN17, RN1 to RN2, RN2 to RN3, RN3 to RN4, RN14 to RN5, RN15 to RN6, RN16 to RN7, RN17 to RN8, RN4 to RN9, U0 to U1, U1 to U2
Connections:
- J1 pad 13: Net-(J0-Pad13) -> (no net)
- J1 pad 14: Net-(J0-Pad14) -> (no net)
- J1 pad 15: Net-(J0-Pad15) -> (no net)
- J1 pad 16: Net-(J0-Pad16) -> (no net)
- J1 pad 19: Net-(J0-Pad19) -> (no net)
- U2 pad 11: Net-(U1-Pad11) -> (no net)
- U2 pad 49: Net-(U1-Pad49) -> (no net)
Routing:
- net +3V3: track 73.5 -> 151.6 mm, vias 35 -> 57
- net /HDMI/DK1: track 28.5 -> 13.1 mm
- net /DIP13: track 26.6 -> 34.0 mm
- net GNDREF: track 115.7 -> 120.3 mm, vias 39 -> 62
- net Net-(RN1-Pad8): track 4.81 -> 1.92 mm
- net Net-(R3-Pad1): track 5.27 -> 6.67 mm, vias 0 -> 1
- net Net-(R1-Pad2): track 2.84 -> 4.21 mm
- net /HDMI/ISEL: track 5.01 -> 3.83 mm
- net Net-(AFF1-Pad3): track 46.6 -> 45.5 mm
- net /HDMI/DK3: track 5.07 -> 6.07 mm
- net Net-(R4-Pad1): track 8.05 -> 7.13 mm
- net /C1: track 76.0 -> 76.9 mm, vias 5 -> 6
- net Net-(JP5-Pad2): track 15.5 -> 14.7 mm
- net /HS: track 19.8 -> 19.2 mm
- net /VS: track 23.1 -> 22.4 mm
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Other:
- board text added: "IO shield + HDMI V4.0"
- board text removed: "ADSEHGAL IO shield + HDMI V4.0"
