File: IO_Shield_W_HDMI/KiCad Project Files/HDMI.kicad_sch (KiCad schematic)
At the start: 17 parts, among them J1 HDMI_A_1.4, U2 TFP410

Commit message: organized files
Parts:
- R1: value 510 -> 510R
Changed lines of the file:
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@@
   (junction (at 201.295 108.585) (diameter 1.016) (color 0 0 0 0))
   (junction (at 203.835 108.585) (diameter 1.016) (color 0 0 0 0))
+  (no_connect (at 188.595 88.9))
+  (no_connect (at 188.595 93.98))
   (no_connect (at 188.595 86.36))
-  (no_connect (at 188.595 88.9))
   (no_connect (at 188.595 96.52))
   (no_connect (at 139.065 129.54))
   (no_connect (at 188.595 81.28))
-  (no_connect (at 188.595 93.98))
   (bus_entry (at 88.9 52.705) (size 2.54 2.54)
     (stroke (width 0.1524) (type solid) (color 0 0 0 0))
@@
       (effects (font (size 1.27 1.27)) (justify left))
     )
-    (property "Value" "510" (id 1) (at 147.955 47.625 90)
+    (property "Value" "510R" (id 1) (at 147.955 47.625 90)
       (effects (font (size 1.27 1.27)) (justify left))
     )
